File: CAD/electronics/lighthouse/lighthouse.sch (KiCad schematic (older format))
At the start: 8 parts, among them J1 Battery, J2 LED, J3 DC Motor, Q1 Q_NPN_Darlington_EBC, SW1 Tilt switch

Commit message: Electronics sent to manufacturer
Parts:
- Q1: footprint Package_TO_SOT_THT:TO-92L -> Package_TO_SOT_THT:TO-92L_Inline_Wide
- SW1: footprint Resistor_THT:R_Axial_DIN0207_L6.3mm_D2.5mm_P15.24mm_Horizontal -> lighthouse:Mercury tilt switch
Changed lines of the file:
@@
 F 0 "SW1" H 1850 2317 50  0000 C CNN
 F 1 "Tilt switch" H 1850 2226 50  0000 C CNN
-F 2 "Resistor_THT:R_Axial_DIN0207_L6.3mm_D2.5mm_P15.24mm_Horizontal" H 1850 2050 50  0001 C CNN
+F 2 "lighthouse:Mercury tilt switch" H 1850 2050 50  0001 C CNN
 F 3 "~" H 1850 2050 50  0001 C CNN
 	1    1850 2050
@@
 F 0 "Q1" H 2840 2096 50  0000 L CNN
 F 1 "Q_NPN_Darlington_EBC" H 2840 2005 50  0000 L CNN
-F 2 "Package_TO_SOT_THT:TO-92L" H 2850 2150 50  0001 C CNN
+F 2 "Package_TO_SOT_THT:TO-92L_Inline_Wide" H 2850 2150 50  0001 C CNN
 F 3 "~" H 2650 2050 50  0001 C CNN
 	1    2650 2050
