File: CAD/electronics/power-supply/power-supply.sch (KiCad schematic (older format))
At the start: 26 parts, among them J1 Batterie, J2 12V, J3 5V servo, U1 LM7805_TO220, U3 LM741, U6 LM2576T-5

Commit message: Electronics sent to manufacturer
Parts:
- removed C1: 330n, Capacitor_THT:C_Rect_L11.0mm_W2.8mm_P10.00mm_MKT, symbol Device:C
- removed C3: 100n, Capacitor_THT:C_Rect_L11.0mm_W2.8mm_P10.00mm_MKT, symbol Device:C
- removed D7: 6V Zener, Diode_THT:D_DO-15_P10.16mm_Horizontal, symbol Device:D_Zener
- removed U1: LM7805_TO220, Package_TO_SOT_THT:TO-220-3_Horizontal_TabDown, symbol Regulator_Linear:LM7805_TO220
- C2: footprint Capacitor_THT:CP_Radial_D10.0mm_P5.00mm -> Capacitor_THT:CP_Radial_D6.3mm_P2.50mm
- C4: footprint Capacitor_THT:CP_Radial_D10.0mm_P7.50mm -> Capacitor_THT:CP_Radial_D10.0mm_P5.00mm
- D1, D2: footprint Diode_THT:D_DO-15_P15.24mm_Horizontal -> Diode_THT:D_P600_R-6_P12.70mm_Horizontal
- L1: footprint Inductor_THT:L_Radial_D12.5mm_P7.00mm_Fastron_09HCP -> Inductor_THT:L_Toroid_Vertical_L54.0mm_W23.8mm_P20.10mm_Bourns_5700
- U6: footprint Package_TO_SOT_THT:TO-220-5_Horizontal_TabDown -> Package_TO_SOT_THT:TO-220-5_Vertical
Connections:
- net 12V: now also A1.8 (VIN)
- no-connect marks 29 -> 28
Other:
- moved on the sheet: C4, D2, J3, L1, U6
