File: robot2/CAD/electrical/main_board/main_board.kicad_pcb (KiCad board)
At the start: 2 copper layers, 85.7 x 55.2 mm, 43 parts, among them J10 I2C Motor, J7 I2C Peripheral, U1 LM2576S-5, U2 AMS1117-3.3, U4 PCA9306DC, U5 PCA9306DC, U6 MPU-6050

Commit message: Main board v2
Parts:
- added R7: 10k, Resistor_SMD:R_1206_3216Metric, F.Cu at (53.6, 58.7)
- added R8: 10k, Resistor_SMD:R_1206_3216Metric, F.Cu at (56.1, 58.7)
- J1: renamed from 12V in
- J2: renamed from Raspberry Pi header
- J8: renamed from I2C periph
- J9: renamed from I2C motor
- R1: value 220 -> 300
- R5, R6: value 200k -> 100k
- U4, U5: value PCA9306DC -> PCA9306DC1
- moved U6 5.30 mm to (82.4, 62.6)
- moved C6 5.30 mm to (85.1, 68.2)
- moved C7 5.30 mm to (79.4, 68.2)
- moved C8 5.24 mm to (83.2, 58.4)
- moved U4 0.90 mm to (109.9, 57.8)
- moved U5 0.63 mm to (109.2, 47.0)
- moved D2 0.13 mm to (43.3, 81.3)
- moved D4 0.13 mm to (43.3, 85.1)
- renumbered JTAG to J11, UART to J12, Trigger to J3, Side to J4, A to J5, B to J6, RESET to SW1, BOOT to SW2, ESP32 to U3
Connections:
- U3 pad 10: /BTN_B -> /SPI2_MOSI
- U3 pad 26: Net-(U3-Pad26) -> /SPI2_CLK
- U3 pad 29: Net-(U3-Pad29) -> /SPI2_CS0
- U3 pad 37: /BTN_A -> /SPI2_MISO
- U3 pad 6: Net-(U3-Pad6) -> /BTN_A
- U3 pad 7: Net-(U3-Pad7) -> /BTN_B
- U4 pad 1: +3V3 -> GND
- U4 pad 2: /SCL_PERIPH -> +3V3
- U4 pad 3: /SDA_PERIPH -> /SCL_PERIPH
- U4 pad 4: GND -> /SDA_PERIPH
- U5 pad 1: +3V3 -> GND
- U5 pad 2: /SCL_MOTOR -> +3V3
- U5 pad 3: /SDA_MOTOR -> /SCL_MOTOR
- U5 pad 4: GND -> /SDA_MOTOR
- U6 pad 23: /SCL_PERIPH -> /SPI2_CLK
- U6 pad 24: /SDA_PERIPH -> /SPI2_MOSI
- U6 pad 8: +3V3 -> /SPI2_CS0
- U6 pad 9: GND -> /SPI2_MISO
Routing:
- net /SPI2_CS0: track 0.00 -> 64.4 mm, vias 0 -> 2
- net /SPI2_MISO: track 0.00 -> 63.2 mm, vias 0 -> 2
- net /SPI2_CLK: track 0.00 -> 55.8 mm, vias 0 -> 2
- net /BTN_A: track 142.5 -> 102.9 mm, vias 2 -> 4
- net /SPI2_MOSI: track 0.00 -> 39.1 mm, vias 0 -> 2
- net /SCL_PERIPH: track 84.2 -> 51.8 mm, vias 2 -> 0
- net /SDA_PERIPH: track 77.2 -> 48.9 mm, vias 2 -> 0
- net /UART_MOSI: track 137.2 -> 119.4 mm
- net /UART_MISO: track 133.3 -> 117.6 mm, vias 1 -> 2
- net +3V3: track 206.4 -> 221.9 mm, vias 2 -> 3
- net GND: track 174.3 -> 164.1 mm, vias 13 -> 14
- net /BTN_B: track 99.6 -> 107.6 mm
- net /JTAG_TMS: track 17.2 -> 19.5 mm
- net Net-(R2-Pad2): track 92.0 -> 90.4 mm
- net /SPI_CLK: track 49.3 -> 50.4 mm
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Other:
- board text added: "A"
- board text added: "B"
- board text added: "Boot"
- board text added: "E.S.C.Ro.C.S 2022 ~ Age of Bots ~"
- board text added: "I2C motor"
- board text added: "I2C peripheral"
- board text added: "JTAG"
- board text added: "Main control board"
- board text added: "Raspberry Pi header"
- board text added: "Reset"
- board text added: "Side"
- board text added: "Trigger"
- board text added: "UART"
