File: CAD/electrical/main_board_v2/usb_uart.kicad_sch (KiCad schematic)
At the start: 17 parts, among them J301 USB_B, J302 UART PGM, Q301 Q_NPN_BEC, Q302 Q_NPN_BEC, SW301 BOOT, SW302 RESET, U301 SRV05-4, U302 CP2102N-Axx-xQFN28

Commit message: Kicad CAD for mainboard and motorboard (final)
Parts:
- removed J302: UART PGM, Connector_Molex:Molex_KK-254_AE-6410-04A_1x04_P2.54mm_Vertical, symbol Connector:Conn_01x04_Male
- R301: value 47k -> 82k
- R302: value 24k -> 47k
- SW301, SW302: footprint Button_Switch_THT:SW_PUSH_6mm -> Button_Switch_SMD:SW_Push_1P1T_NO_6x6mm_H9.5mm
Connections:
- no-connect marks 19 -> 18
Changed lines of the file:
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@@
   (junction (at 170.18 85.09) (diameter 0) (color 0 0 0 0)
-  )
-  (junction (at 170.18 149.86) (diameter 0) (color 0 0 0 0)
   )
   (junction (at 88.9 149.86) (diameter 0) (color 0 0 0 0)
@@
   (no_connect (at 153.67 110.49))
   (no_connect (at 153.67 80.01))
-  (no_connect (at 167.64 116.84))
   (no_connect (at 153.67 125.73))
   (no_connect (at 153.67 95.25))
@@
     (stroke (width 0) (type default) (color 0 0 0 0))
   )
-  (wire (pts (xy 140.97 149.86) (xy 170.18 149.86))
-    (stroke (width 0) (type default) (color 0 0 0 0))
-  )
   (wire (pts (xy 190.5 80.01) (xy 190.5 81.28))
     (stroke (width 0) (type default) (color 0 0 0 0))
@@
     (stroke (width 0) (type default) (color 0 0 0 0))
   )
-  (wire (pts (xy 170.18 149.86) (xy 190.5 149.86))
+  (wire (pts (xy 140.97 149.86) (xy 190.5 149.86))
     (stroke (width 0) (type default) (color 0 0 0 0))
   )
@@
     (stroke (width 0) (type default) (color 0 0 0 0))
   )
-  (wire (pts (xy 170.18 124.46) (xy 167.64 124.46))
-    (stroke (width 0) (type default) (color 0 0 0 0))
-  )
   (wire (pts (xy 190.5 97.79) (xy 199.39 97.79))
     (stroke (width 0) (type default) (color 0 0 0 0))
@@
   )
   (wire (pts (xy 125.73 129.54) (xy 125.73 100.33))
-    (stroke (width 0) (type default) (color 0 0 0 0))
-  )
-  (wire (pts (xy 170.18 149.86) (xy 170.18 124.46))
     (stroke (width 0) (type default) (color 0 0 0 0))
   )
@@
     (effects (font (size 1.27 1.27)) (justify left))
   )
-  (hierarchical_label "RX" (shape input) (at 167.64 121.92 0)
-    (effects (font (size 1.27 1.27)) (justify left))
-  )
   (hierarchical_label "RX" (shape input) (at 153.67 74.93 0)
-    (effects (font (size 1.27 1.27)) (justify left))
-  )
-  (hierarchical_label "TX" (shape output) (at 167.64 119.38 0)
     (effects (font (size 1.27 1.27)) (justify left))
   )
@@
       (effects (font (size 1.27 1.27)) (justify right))
     )
-    (property "Footprint" "Button_Switch_THT:SW_PUSH_6mm" (id 2) (at 190.5 59.69 0)
+    (property "Footprint" "Button_Switch_SMD:SW_Push_1P1T_NO_6x6mm_H9.5mm" (id 2) (at 190.5 59.69 0)
       (effects (font (size 1.27 1.27)) hide)
     )
@@
     (pin "9")
   )
-  (symbol (lib_id "Connector:Conn_01x04_Male") (at 162.56 119.38 0) (unit 1)
-    (in_bom yes) (on_board yes)
-    (property "Reference" "J302" (id 0) (at 165.3032 112.2426 0))
-    (property "Value" "UART PGM" (id 1) (at 165.3032 114.554 0))
-    (property "Footprint" "Connector_Molex:Molex_KK-254_AE-6410-04A_1x04_P2.54mm_Vertical" (id 2) (at 162.56 119.38 0)
-      (effects (font (size 1.27 1.27)) hide)
-    )
-    (property "Datasheet" "~" (id 3) (at 162.56 119.38 0)
-      (effects (font (size 1.27 1.27)) hide)
-    )
-    (pin "1")
-    (pin "2")
-    (pin "3")
-    (pin "4")
-  )
   (symbol (lib_id "Device:Q_NPN_BEC") (at 187.96 74.93 0) (unit 1)
     (in_bom yes) (on_board yes) (fields_autoplaced)
@@
       (effects (font (size 1.27 1.27)) (justify right))
     )
-    (property "Footprint" "Button_Switch_THT:SW_PUSH_6mm" (id 2) (at 190.5 105.41 0)
+    (property "Footprint" "Button_Switch_SMD:SW_Push_1P1T_NO_6x6mm_H9.5mm" (id 2) (at 190.5 105.41 0)
       (effects (font (size 1.27 1.27)) hide)
     )
@@
   (symbol (lib_id "Device:R") (at 114.3 80.01 180) (unit 1)
     (in_bom yes) (on_board yes) (fields_autoplaced)
-    (property "Reference" "R301" (id 0) (at 118.11 78.7399 0)
-      (effects (font (size 1.27 1.27)) (justify right))
-    )
-    (property "Value" "47k" (id 1) (at 118.11 81.2799 0)
+    (property "Reference" "R301" (id 0) (at 116.84 78.7399 0)
+      (effects (font (size 1.27 1.27)) (justify right))
+    )
+    (property "Value" "82k" (id 1) (at 116.84 81.2799 0)
       (effects (font (size 1.27 1.27)) (justify right))
     )
@@
   (symbol (lib_id "Device:R") (at 114.3 90.17 180) (unit 1)
     (in_bom yes) (on_board yes) (fields_autoplaced)
-    (property "Reference" "R302" (id 0) (at 118.11 88.8999 0)
-      (effects (font (size 1.27 1.27)) (justify right))
-    )
-    (property "Value" "24k" (id 1) (at 118.11 91.4399 0)
-      (effects (font (size 1.27 1.27)) (justify right))
-    )
+    (property "Reference" "R302" (id 0) (at 116.84 88.8999 0)
+      (effects (font (size 1.27 1.27)) (justify right))
+    )
+    (property "Value" "47k" (id 1) (at 116.84 91.4399 0)
+      (effects (font (size 1.27 1.27)) (justify right))
+    )

Commit message: LD06 board colplet
Parts:
- R307, R308: LCSC (none) -> C22775
