File: CAD/electrical/accessory_board/accessory_board.kicad_pcb (KiCad board)
At the start: 2 copper layers, 123.2 x 55.2 mm, 61 parts, among them J1 Battery in, J10 Servo 0, J11 Servo 1, J12 Servo 2, J13 Servo 3, J14 Servo 4, J15 Servo 5, J16 Servo 6, J17 Servo 7, J18 Servo A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

Commit message: update ld06 I2C for button
Other:
- net class Default removed
- net class Power removed
